File: Hardware/SparkFun_Mini_GPS_Shield.brd (EAGLE design)
At the start: 17.8 x 34.3 mm, 19 parts, among them J1 MICROSD_TINY, U1 GP735, U2 TXB0108, U3 AP2112K-3.3V

Commit message: V10 Changes
- Changed board name to "Mini GPS Shield".
- Extended board length to better support uSD card.
- Added v-score to board extention
- Changed control pin name to "CTL" instead of "CTR"
Parts:
- moved LOGO1 6.96 mm to (7.37, 10.3), turned to 90 degrees
- moved C6 5.72 mm to (5.08, 16.5)
- moved U3 5.72 mm to (4.95, 19.4)
- moved J2 5.72 mm to (1.27, 8.26)
- moved J3 5.72 mm to (16.5, 8.26)
- moved C5 5.71 mm to (4.95, 22.7)
- moved D1 5.71 mm to (4.19, 31.4)
- moved FD1 5.71 mm to (2.54, 6.99)
- moved J1 5.71 mm to (3.30, 8.13)
- moved J5 5.71 mm to (6.60, 28.2)
- moved LOGO3 5.71 mm to (11.4, 15.5)
- moved LOGO4 5.71 mm to (6.60, 23.5)
- moved R1 5.71 mm to (4.19, 28.1)
- moved S1 5.71 mm to (11.2, 27.1)
- moved U1 5.71 mm to (11.4, 34.3)
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Other:
- board size 17.8 x 34.3 mm -> 17.8 x 40 mm
- board text added: "CTL"
- board text added: "Mini GPS Shield"
- board text added: "V-score"
- board text added: "v10"
- board text removed: "CTR"
- board text removed: "Pro Mini GPS Shield"
- board text removed: "v01"
