File: Hardware/SparkFun_Mini_GPS_Shield.brd (EAGLE design)
At the start: 17.8 x 40 mm, 19 parts, among them J1 MICROSD_TINY, U1 GP735, U2 TXB0108, U3 AP2112K-3.3V

Commit message: Changed UART net labels
0/RX and 1/TX are now RX/0 and TX/1
Connections:
- net 0/RX renamed RX/0
- net 1/TX renamed TX/1
Changed lines of the file:
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@@
 <?xml version="1.0" encoding="utf-8"?>
 <!DOCTYPE eagle SYSTEM "eagle.dtd">
-<eagle version="7.6.0">
+<eagle version="7.7.0">
 <drawing>
 <settings>
@@
 <layer number="20" name="Dimension" color="15" fill="1" visible="yes" active="yes"/>
 <layer number="21" name="tPlace" color="16" fill="1" visible="yes" active="yes"/>
-<layer number="22" name="bPlace" color="14" fill="1" visible="no" active="yes"/>
+<layer number="22" name="bPlace" color="14" fill="1" visible="yes" active="yes"/>
 <layer number="23" name="tOrigins" color="15" fill="1" visible="yes" active="yes"/>
-<layer number="24" name="bOrigins" color="15" fill="1" visible="no" active="yes"/>
+<layer number="24" name="bOrigins" color="15" fill="1" visible="yes" active="yes"/>
 <layer number="25" name="tNames" color="7" fill="1" visible="no" active="yes"/>
 <layer number="26" name="bNames" color="7" fill="1" visible="no" active="yes"/>
@@
 <layer number="43" name="vRestrict" color="2" fill="10" visible="no" active="yes"/>
 <layer number="44" name="Drills" color="7" fill="1" visible="no" active="yes"/>
-<layer number="45" name="Holes" color="7" fill="1" visible="no" active="yes"/>
+<layer number="45" name="Holes" color="7" fill="1" visible="yes" active="yes"/>
 <layer number="46" name="Milling" color="3" fill="1" visible="no" active="yes"/>
 <layer number="47" name="Measures" color="7" fill="1" visible="yes" active="yes"/>
@@
 <wire x1="8.255" y1="12.319" x2="8.255" y2="10.3032" width="0.254" layer="1"/>
 </signal>
-<signal name="1/TX">
+<signal name="TX/1">
 <contactref element="J2" pad="12"/>
 <contactref element="S1" pad="6"/>
@@
 <wire x1="12.486" y1="29.551" x2="11.938" y2="30.099" width="0.254" layer="1"/>
 </signal>
-<signal name="0/RX">
+<signal name="RX/0">
 <contactref element="J2" pad="11"/>
 <contactref element="S1" pad="3"/>
